File: ECU-Designs/Motor controller adapter board/Motor Controller removable maintenance adapter board.sch (EAGLE design)
At the start: 5 parts, among them X1 MINIFIT_5566-6

Commit message: Updated moter controller board with switch designation
Parts:
- R1: device HyTechDevices:RESISTOR0402 -> HyTechDevices:RESISTOR0805-RES
Changed lines of the file:
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@@
 <part name="X1" library="HyTechDevices" deviceset="MINIFIT_5566-6" device=""/>
 <part name="LED1" library="HyTechDevices" deviceset="LED" device="-0805"/>
-<part name="R1" library="HyTechDevices" deviceset="RESISTOR" device="0402"/>
+<part name="R1" library="HyTechDevices" deviceset="RESISTOR" device="0805-RES"/>
 <part name="GND1" library="HyTechSymbols" deviceset="GND" device=""/>
 <part name="X2" library="con-subd" deviceset="F09HP" device=""/>
